Commit message: found a bunch of silly kinematics errors

File: legup/robots/mini_cheetah/physical_models/mini-cheetah.urdf (robot description, URDF)
Before this commit: robot mini_cheetah, 13 links, 12 joints
Joints:
- joint abduct_fl_to_thigh_fl_j: axis 0 -1 0 -> 0 1 0
- joint abduct_hl_to_thigh_hl_j: axis 0 -1 0 -> 0 1 0
- joint thigh_fl_to_knee_fl_j: axis 0 -1 0 -> 0 1 0
- joint thigh_hl_to_knee_hl_j: axis 0 -1 0 -> 0 1 0
